File: pcb/tt-i2c-jr.brd (EAGLE design)
At the start: 35.6 x 23.2 mm, 9 parts

Commit message: updated board files/dxf
Parts:
- U$1: value ADP3339 -> AZ1117CH-3.3TRG1DICT-ND
- moved U$2 0.63 mm to (51.4, 12.1)
- moved U$3 0.32 mm to (79.4, 13.0)
Other:
- outline, holes or cut-outs redrawn
- board text added: "tt-busboard-jr by steven noreyko/denki_oto january 2019 adapted from Teletype Busboard by Brian Crabtree"
Changed lines of the file:
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@@
 <?xml version="1.0" encoding="utf-8"?>
 <!DOCTYPE eagle SYSTEM "eagle.dtd">
-<eagle version="9.1.3">
+<eagle version="9.2.2">
 <drawing>
 <settings>
@@
 <setting verticaltext="up"/>
 </settings>
-<grid distance="0.05" unitdist="inch" unit="inch" style="dots" multiple="1" display="yes" altdistance="0.0125" altunitdist="inch" altunit="inch"/>
+<grid distance="0.05" unitdist="inch" unit="mil" style="dots" multiple="1" display="yes" altdistance="0.0125" altunitdist="inch" altunit="mil"/>
 <layers>
 <layer number="1" name="Top" color="4" fill="1" visible="yes" active="yes"/>
@@
 <layer number="20" name="Dimension" color="15" fill="1" visible="yes" active="yes"/>
 <layer number="21" name="tPlace" color="7" fill="1" visible="yes" active="yes"/>
-<layer number="22" name="bPlace" color="7" fill="1" visible="no" active="yes"/>
+<layer number="22" name="bPlace" color="7" fill="1" visible="yes" active="yes"/>
 <layer number="23" name="tOrigins" color="15" fill="1" visible="yes" active="yes"/>
 <layer number="24" name="bOrigins" color="15" fill="1" visible="yes" active="yes"/>
 <layer number="25" name="tNames" color="7" fill="1" visible="yes" active="yes"/>
 <layer number="26" name="bNames" color="7" fill="1" visible="yes" active="yes"/>
-<layer number="27" name="tValues" color="7" fill="1" visible="no" active="yes"/>
-<layer number="28" name="bValues" color="7" fill="1" visible="no" active="yes"/>
+<layer number="27" name="tValues" color="7" fill="1" visible="yes" active="yes"/>
+<layer number="28" name="bValues" color="7" fill="1" visible="yes" active="yes"/>
 <layer number="29" name="tStop" color="7" fill="3" visible="no" active="yes"/>
 <layer number="30" name="bStop" color="7" fill="6" visible="no" active="yes"/>
@@
 <text x="49.2125" y="5.3975" size="1.27" layer="21" ratio="12">SCL</text>
 <text x="49.2125" y="2.8575" size="1.27" layer="21" ratio="12">SDA</text>
-<text x="63.5" y="16.51" size="1.27" layer="21" ratio="12" rot="R90">-12V</text>
-<wire x1="48.26" y1="23.1775" x2="83.82" y2="23.1775" width="0" layer="20"/>
-<wire x1="83.82" y1="23.1775" x2="83.82" y2="0" width="0" layer="20"/>
-<wire x1="83.82" y1="0" x2="48.26" y2="0" width="0" layer="20"/>
-<wire x1="48.26" y1="0" x2="48.26" y2="6.35" width="0" layer="20"/>
-<wire x1="48.26" y1="6.35" x2="48.26" y2="23.1775" width="0" layer="20"/>
+<text x="62.865" y="16.51" size="1.27" layer="21" ratio="12" rot="R90">-12V</text>
+<wire x1="48.26" y1="6.35" x2="48.26" y2="21.9075" width="0" layer="20"/>
+<wire x1="48.26" y1="21.9075" x2="49.53" y2="23.1775" width="0" layer="20" curve="-90"/>
+<wire x1="49.53" y1="23.1775" x2="82.55" y2="23.1775" width="0" layer="20"/>
+<wire x1="82.55" y1="23.1775" x2="83.82" y2="21.9075" width="0" layer="20" curve="-90"/>
+<wire x1="83.82" y1="21.9075" x2="83.82" y2="1.27" width="0" layer="20"/>
+<wire x1="83.82" y1="1.27" x2="82.55" y2="0" width="0" layer="20" curve="-90"/>
+<wire x1="82.55" y1="0" x2="49.53" y2="0" width="0" layer="20"/>
+<wire x1="49.53" y1="0" x2="48.26" y2="1.27" width="0" layer="20" curve="-90"/>
+<wire x1="48.26" y1="1.27" x2="48.26" y2="6.35" width="0" layer="20"/>
 <text x="49.2125" y="7.9375" size="1.27" layer="21" ratio="12">GND</text>
 <rectangle x1="53.34" y1="20.32" x2="60.96" y2="22.225" layer="22"/>
 <rectangle x1="53.34" y1="7.62" x2="60.96" y2="9.525" layer="21" rot="R180"/>
-<rectangle x1="63.8175" y1="14.9225" x2="67.945" y2="22.5425" layer="21" rot="R180"/>
+<rectangle x1="63.1825" y1="14.9225" x2="67.31" y2="22.5425" layer="21" rot="R180"/>
 <text x="80.9625" y="10.4775" size="0.6096" layer="21" ratio="12">GND</text>
 <text x="80.9625" y="1.5875" size="0.6096" layer="21" ratio="12">SDA</text>
@@
 <text x="49.2125" y="15.5575" size="1.27" layer="21" ratio="12">SDA</text>
 <text x="49.2125" y="20.6375" size="1.27" layer="21" ratio="12">GND</text>
-<text x="66.04" y="1.27" size="0.6096" layer="25">2.2K</text>
-<text x="66.04" y="7.62" size="0.6096" layer="25">2.2K</text>
+<text x="63.5" y="1.27" size="0.6096" layer="25">2.2K</text>
+<text x="63.5" y="7.9375" size="0.6096" layer="25">2.2K</text>
 <rectangle x1="53.34" y1="20.32" x2="60.96" y2="22.225" layer="21" rot="R180"/>
 <rectangle x1="75.8825" y1="7.9375" x2="83.5025" y2="9.8425" layer="21" rot="R180"/>
 <rectangle x1="53.34" y1="7.62" x2="60.96" y2="9.525" layer="22"/>
 <rectangle x1="53.34" y1="7.62" x2="60.96" y2="9.525" layer="21" rot="R180"/>
+<text x="55.245" y="11.7475" size="0.4064" layer="21">tt-busboard-jr by steven noreyko/denki_oto
+january 2019
+adapted from Teletype Busboard by Brian Crabtree</text>
 </plain>
 <attributes>
@@
 </autorouter>
 <elements>
-<element name="U$1" library="monome-inc" package="SOT223" value="ADP3339" x="71.755" y="6.0325" smashed="yes" rot="R270">
-<attribute name="VALUE" x="66.04" y="8.5725" size="0.8128" layer="27" ratio="10" rot="R270"/>
+<element name="U$1" library="monome-inc" package="SOT223" value="AZ1117CH-3.3TRG1DICT-ND" x="71.755" y="6.0325" smashed="yes" rot="R270">
+<attribute name="VALUE" x="72.39" y="9.525" size="0.4064" layer="27" ratio="10" rot="R270"/>
 </element>
-<element name="R5" library="rc-master-smd" package="R1206" value="2k2" x="64.135" y="3.4925" smashed="yes">
-<attribute name="VALUE" x="62.865" y="1.7462" size="0.8128" layer="27" ratio="10"/>
-</element>
-<element name="R16" library="rc-master-smd" package="R1206" value="2k2" x="64.135" y="6.0325" smashed="yes">
-<attribute name="VALUE" x="62.865" y="4.2862" size="0.8128" layer="27" ratio="10"/>
-</element>
+<element name="R5" library="rc-master-smd" package="R1206" value="2k2" x="64.135" y="3.4925" smashed="yes"/>
+<element name="R16" library="rc-master-smd" package="R1206" value="2k2" x="64.135" y="6.0325" smashed="yes"/>
 <element name="JP11" library="pinhead" package="2X05" value="" x="73.025" y="18.7325" smashed="yes">
 <attribute name="VALUE" x="66.675" y="14.2875" size="1.27" layer="27"/>
@@
 <attribute name="VALUE" x="75.565" y="10.16" size="1.27" layer="27" rot="R270"/>
 </element>
-<element name="U$2" library="microbuilder" package="MOUNTINGHOLE_3.0_PLATEDTHIN" value="MOUNTINGHOLE3.0THIN" x="51.435" y="11.43"/>
-<element name="U$3" library="microbuilder" package="MOUNTINGHOLE_3.0_PLATEDTHIN" value="MOUNTINGHOLE3.0THIN" x="79.375" y="13.335"/>
+<element name="U$2" library="microbuilder" package="MOUNTINGHOLE_3.0_PLATEDTHIN" value="MOUNTINGHOLE3.0THIN" x="51.435" y="12.065" smashed="yes"/>
+<element name="U$3" library="microbuilder" package="MOUNTINGHOLE_3.0_PLATEDTHIN" value="MOUNTINGHOLE3.0THIN" x="79.375" y="13.0175" smashed="yes"/>
 </elements>
 <signals>
@@
 <contactref element="JP11" pad="7"/>
 <polygon width="0.4064" layer="16">
-<vertex x="48.26" y="0"/>
-<vertex x="48.26" y="23.1775"/>
-<vertex x="83.82" y="23.1775"/>
-<vertex x="83.82" y="0"/>
+<vertex x="48.5775" y="0.3175"/>
+<vertex x="48.5775" y="22.86"/>
+<vertex x="83.185" y="22.86"/>
+<vertex x="83.185" y="0.3175"/>
 </polygon>
 <contactref element="JP15" pad="2"/>
@@
 </board>
 </drawing>
+<compatibility>
+<note version="6.3" minversion="6.2.2" severity="warning">
+Since Version 6.2.2 text objects can contain more than one line,
+which will not be processed correctly with this version.
+</note>
+</compatibility>
 </eagle>
